Commit message: 11/05

File: src/ur3_project/urdf/gripper.urdf.xacro (robot description, xacro)
@@ -61,6 +61,6 @@
     </link>
     <joint name="${prefix}gripper_base_joint" type="fixed">
-      <!-- -90 deg about end-effector Z aligns fingers with the camera orientation -->
-      <origin xyz="0 0 0" rpy="0 0 -1.5707963"/>
+      <!-- -180 + 25 = -155 deg about end-effector Z (matches real robot mounting) -->
+      <origin xyz="0 0 0" rpy="0 0 -2.7052604"/>
       <parent link="${parent}"/>
       <child  link="${prefix}gripper_base_link"/>

File: src/ur3_project/urdf/ur.ros2_control.xacro (robot description, xacro)
@@ -138,22 +138,4 @@
         <state_interface name="effort"/>
       </joint>
-      <!-- Gripper finger joints — always included when include_gripper is set,
-           regardless of sim or fake-hardware mode. -->
-      <xacro:if value="${include_gripper}">
-        <joint name="gripper_left_finger_joint">
-          <command_interface name="position"/>
-          <state_interface name="position">
-            <param name="initial_value">0.02</param>
-          </state_interface>
-          <state_interface name="velocity"/>
-        </joint>
-        <joint name="gripper_right_finger_joint">
-          <command_interface name="position"/>
-          <state_interface name="position">
-            <param name="initial_value">0.02</param>
-          </state_interface>
-          <state_interface name="velocity"/>
-        </joint>
-      </xacro:if>
       <xacro:unless value="${sim_gazebo or sim_ignition}">
         <sensor name="${tf_prefix}tcp_fts_sensor">
@@ -372,4 +354,31 @@
       </xacro:unless>
     </ros2_control>
+    <!-- Gripper finger joints in a separate ros2_control block so they are
+         never passed to URPositionHardwareInterface, which only handles the
+         6 UR arm joints. mock_components/GenericSystem acts as a passthrough
+         (commands echoed back as state) regardless of real/fake/sim mode. -->
+    <xacro:if value="${include_gripper}">
+      <ros2_control name="gripper" type="system">
+        <hardware>
+          <plugin>mock_components/GenericSystem</plugin>
+          <param name="fake_sensor_commands">false</param>
+          <param name="state_following_offset">0.0</param>
+        </hardware>
+        <joint name="gripper_left_finger_joint">
+          <command_interface name="position"/>
+          <state_interface name="position">
+            <param name="initial_value">0.02</param>
+          </state_interface>
+          <state_interface name="velocity"/>
+        </joint>
+        <joint name="gripper_right_finger_joint">
+          <command_interface name="position"/>
+          <state_interface name="position">
+            <param name="initial_value">0.02</param>
+          </state_interface>
+          <state_interface name="velocity"/>
+        </joint>
+      </ros2_control>
+    </xacro:if>
   </xacro:macro>
 </robot>

File: src/ur3_project/urdf/ur3.srdf.xacro (robot description, xacro)
@@ -5,15 +5,16 @@
     <chain base_link="base_link" tip_link="gripper_tcp_link"/>
   </group>
-  <!-- wait_forward: gripper_tcp_link at WAIT_TCP (0.30, 0.20, 0.35), facing +Y
-       (FORWARD_QUAT = (0, 0.7071, 0.7071, 0)). wrist_3 = +pi/2 branch, shared
+  <!-- wait_forward: gripper_tcp_link at WAIT_TCP (0.20, -0.30, 0.26) in base_link
+       (= world (0.30, 0.20, 1.06)), facing +X in base_link / +Y in world
+       (FORWARD_QUAT = (0.5, 0.5, 0.5, 0.5)). wrist_3 = +pi branch, shared
        by all pick-cycle IK solutions so no 2*pi joint jump occurs. Joint values
        below match config/initial_positions.yaml so spawn lands here. -->
   <group_state name="wait_forward" group="ur_manipulator">
-    <joint name="shoulder_pan_joint"  value="0.2210"/>
+    <joint name="shoulder_pan_joint"  value="4.9333890"/>
     <joint name="shoulder_lift_joint" value="-2.2994"/>
     <joint name="elbow_joint"         value="1.8025"/>
     <joint name="wrist_1_joint"       value="0.4969"/>
     <joint name="wrist_2_joint"       value="0.2210"/>
-    <joint name="wrist_3_joint"       value="1.5708"/>
+    <joint name="wrist_3_joint"       value="2.7052640"/>
   </group_state>
   <!-- home: legacy forward-facing pose at (0.418, 0.112, 0.402). wrist_3=+pi branch.

File: src/ur3_project/urdf/ur3_camera_gripper.urdf.xacro (robot description, xacro)
@@ -115,5 +115,5 @@
     trajectory_port="$(arg trajectory_port)"
     >
-    <origin xyz="0 0 0.8" rpy="0 0 0"/>
+    <origin xyz="0 0 0.8" rpy="0 0 ${pi/2}"/>
   </xacro:ur_robot>
   <!-- ════════════════════════════════════════════════════════════════════
