Commit message: Fixed grasping and implemented vision

File: src/ur3_project/urdf/camera.urdf.xacro (robot description, xacro)
@@ -59,5 +59,5 @@
     <parent link="gripper_base_link"/>
     <child  link="camera_link"/>
-    <origin xyz="0 0.050 0.095" rpy="0 -1.5707963 -1.5707963"/>
+    <origin xyz="-0.09 0.115 0.025" rpy="1.5707963 -1.5707963 -1.5707963"/>
   </joint>
   <!-- ── Optical frame ────────────────────────────────────────────────── -->

Commit message: New YOLO Model

File: src/ur3_project/urdf/camera.urdf.xacro (robot description, xacro)
@@ -43,9 +43,6 @@
       <material name="camera_red"/>
     </visual>
-    <collision>
-      <geometry>
-        <mesh filename="package://ur3_project/meshes/sensors/camera/kinetic.dae"/>
-      </geometry>
-    </collision>
+    <!-- Camera collision disabled for testing — re-enable once the
+         identify-pose / forward orientation passes without false hits. -->
   </link>
   <!--
@@ -59,5 +56,5 @@
     <parent link="gripper_base_link"/>
     <child  link="camera_link"/>
-    <origin xyz="-0.09 0.115 0.025" rpy="1.5707963 -1.5707963 -1.5707963"/>
+    <origin xyz="-0.09 0.065 0.025" rpy="1.5707963 -1.5707963 -1.5707963"/>
   </joint>
   <!-- ── Optical frame ────────────────────────────────────────────────── -->

File: src/ur3_project/urdf/gripper.urdf.xacro (robot description, xacro)
@@ -30,25 +30,30 @@
   Midpoint of the gripping zone: Z = 0.120 m (base) + 0.053 m (½ finger length)
                                     = 0.173 m from tool0
+  This is the single source of truth for the gripper TCP. The Python IK
+  chain in pick_place_manager_node.py mirrors it in TCP_Z_OFFSET — keep
+  the two in sync.
 -->
 <robot xmlns:xacro="http://wiki.ros.org/xacro">
   <xacro:macro name="parallel_gripper" params="prefix parent *origin">
     <!-- ════════════════════════════════════════════════════════════════
-         GRIPPER BASE  (adapter plate, 80 × 80 × 30 mm)
+         GRIPPER BASE  (adapter cylinder, Ø 70 × 100 mm)
+         Extends along gripper_base_link +Z (= TCP direction),
+         0 → 0.100 m. Sits just inside the UR3e wrist_3 flange (radius
+         0.045 m) and reaches up toward the fingers.
          ════════════════════════════════════════════════════════════════ -->
     <link name="${prefix}gripper_base_link">
       <inertial>
-        <origin xyz="0 0 0.015" rpy="0 0 0"/>
+        <origin xyz="0 0 0.050" rpy="0 0 0"/>
         <mass value="0.200"/>
-        <!-- Box 0.080 × 0.080 × 0.030 m, m = 0.200 kg
-             Ixx = (1/12)*0.2*(0.08²+0.03²) = 1.217e-4
-             Iyy = same (square cross-section)
-             Izz = (1/12)*0.2*(0.08²+0.08²) = 2.133e-4 -->
-        <inertia ixx="1.217e-4" ixy="0" ixz="0"
-                 iyy="1.217e-4"       iyz="0"
-                 izz="2.133e-4"/>
+        <!-- Cylinder r=0.035 m, h=0.100 m, m=0.200 kg
+             Ixx = Iyy = (1/12)*m*(3r²+h²) = 2.279e-4
+             Izz       = (1/2)*m*r²        = 1.225e-4 -->
+        <inertia ixx="2.279e-4" ixy="0" ixz="0"
+                 iyy="2.279e-4"       iyz="0"
+                 izz="1.225e-4"/>
       </inertial>
       <visual>
-        <origin xyz="0 0 0.015" rpy="0 0 0"/>
-        <geometry><box size="0.080 0.080 0.030"/></geometry>
+        <origin xyz="0 0 0.050" rpy="0 0 0"/>
+        <geometry><cylinder radius="0.035" length="0.100"/></geometry>
         <material name="${prefix}gripper_aluminium">
           <color rgba="0.75 0.75 0.75 1.0"/>
@@ -56,6 +61,6 @@
       </visual>
       <collision>
-        <origin xyz="0 0 0.015" rpy="0 0 0"/>
-        <geometry><box size="0.080 0.080 0.030"/></geometry>
+        <origin xyz="0 0 0.050" rpy="0 0 0"/>
+        <geometry><cylinder radius="0.035" length="0.100"/></geometry>
       </collision>
     </link>
@@ -156,5 +161,12 @@
     <!-- ════════════════════════════════════════════════════════════════
          TCP  — Tool Centre Point
-         Z = 0.120 m (base height) + 0.053 m (½ finger length) = 0.173 m from tool0
+         Z = 0.120 m (gripper_base_link → finger joint origin)
+           + 0.053 m (½ finger length, 106 mm total)
+           = 0.173 m from tool0
+         This is the geometric midpoint of the finger volume and is where
+         a can sits when fully grasped. If you re-measure the real gripper
+         and need to retune, update this number AND the matching
+         TCP_Z_OFFSET constant in src/pick_place_manager_node.py
+         (they must stay in sync).
          ════════════════════════════════════════════════════════════════ -->
     <link name="${prefix}gripper_tcp_link"/>

File: src/ur3_project/urdf/ur3_camera_gripper.urdf.xacro (robot description, xacro)
@@ -8,6 +8,8 @@
   <xacro:include filename="$(find ur3_project)/urdf/camera.urdf.xacro"/>
   <!-- ── UR robot parameters ──────────────────────────────────────────── -->
-  <!-- possible 'ur_type' values: ur3, ur5, ur10, ur3e, ur5e, … -->
-  <xacro:arg name="ur_type"                  default="ur3"/>
+  <!-- possible 'ur_type' values: ur3, ur5, ur10, ur3e, ur5e, …
+       This project targets the UR3e: link lengths d4/d6 differ from the
+       UR3 by 1–2 cm and the robot calibration YAML is UR3e-extracted. -->
+  <xacro:arg name="ur_type"                  default="ur3e"/>
   <xacro:arg name="tf_prefix"                default=""/>
   <xacro:arg name="joint_limit_params"       default="$(find ur_description)/config/$(arg ur_type)/joint_limits.yaml"/>
